Commit message: check

File: src/my_robot_description/urdf/common_properties.xacro (robot description, xacro)
@@ -8,3 +8,30 @@
         <color rgba="0.5 0.5 0.5 1" />
     </material>
+    <xacro:macro name="box_inertia" params="m l w h xyz rpy">
+        <inertial>
+            <origin xyz="${xyz}" rpy="${rpy}" />
+            <mass value="${m}" />
+            <inertia ixx="${1/12*m*(h*h + l*l)}" ixy="0" ixz="0"
+                     iyy="${m/12*(w*w + l*l)}" iyz="0"
+                     izz="${m/12*(w*w + h*h)}" />
+        </inertial>
+    </xacro:macro>
+    <xacro:macro name="cylinder_inertia" params="m r l xyz rpy">
+        <inertial>
+            <origin xyz="${xyz}" rpy="${rpy}" />
+            <mass value="${m}" />
+            <inertia ixx="${m/12*(3*r*r + l*l)}" ixy="0" ixz="0"
+                     iyy="${m/12*(3*r*r + l*l)}" iyz="0"
+                     izz="${m/12*(r*r)}" />
+        </inertial>
+    </xacro:macro>
+    <xacro:macro name="sphere_inertia" params="m r xyz rpy">
+        <inertial>
+            <origin xyz="${xyz}" rpy="${rpy}" />
+            <mass value="${m}" />
+            <inertia ixx="${2/5*m*r*r}" ixy="0" ixz="0"
+                     iyy="${2/5*m*r*r)}" iyz="0"
+                     izz="${2/5*m*r*r}" />
+        </inertial>
+    </xacro:macro>
 </robot>

File: src/my_robot_description/urdf/mobile_base.xacro (robot description, xacro)
@@ -15,4 +15,6 @@
             <material name="blue" />
         </visual>
+        <xacro:box_inertia m="5.0" l="${base_length}" w="base_width" h="base_height"
+                           xyz="0 0 ${base_height/2.0}" rpy="0 0 0" />
     </link>
     <xacro:macro name="wheel_link" params="prefix">
@@ -25,4 +27,6 @@
                 <material name="grey" />
             </visual>
+            <xacro:box_inertia m="1.0" r="${wheel_radius}" l="wheel_length"
+                            xyz="0 0 0" rpy="${pi/2.0} 0 0" />
         </link>
     </xacro:macro>
@@ -32,9 +36,11 @@
         <visual>
             <geometry>
-                <sphere radius="${wheel_radius/2}" />
+                <sphere radius="${wheel_radius/2.0}" />
             </geometry>
             <origin xyz="0 0 0" rpy="0 0 0" />
             <material name="grey" />
         </visual>
+        <xacro:box_inertia m="0.5" r="${wheel_radius/2.0}"
+                xyz="0 0 0" rpy="0 0 0" />
     </link>
     <joint name="base_joint" type="fixed">

Commit message: bitti

File: src/my_robot_description/urdf/common_properties.xacro (robot description, xacro)
@@ -12,6 +12,6 @@
             <origin xyz="${xyz}" rpy="${rpy}" />
             <mass value="${m}" />
-            <inertia ixx="${1/12*m*(h*h + l*l)}" ixy="0" ixz="0"
-                     iyy="${m/12*(w*w + l*l)}" iyz="0"
+            <inertia ixx="${(m/12) * (h*h + l*l)}" ixy="0" ixz="0"
+                     iyy="${(m/12) * (w*w + l*l)}" iyz="0"
                      izz="${m/12*(w*w + h*h)}" />
         </inertial>
@@ -30,7 +30,7 @@
             <origin xyz="${xyz}" rpy="${rpy}" />
             <mass value="${m}" />
-            <inertia ixx="${2/5*m*r*r}" ixy="0" ixz="0"
-                     iyy="${2/5*m*r*r)}" iyz="0"
-                     izz="${2/5*m*r*r}" />
+            <inertia ixx="${(2/5) * m * r * r}" ixy="0" ixz="0"
+                     iyy="${(2/5)*m*r*r}" iyz="0"
+                     izz="${(2/5)*m*r*r}" />
         </inertial>
     </xacro:macro>

File: src/my_robot_description/urdf/mobile_base.xacro (robot description, xacro)
@@ -15,5 +15,12 @@
             <material name="blue" />
         </visual>
-        <xacro:box_inertia m="5.0" l="${base_length}" w="base_width" h="base_height"
+        <collision>
+            <geometry>
+                <box size="${base_length} ${base_width} ${base_height}" />
+            </geometry>
+            <origin xyz="0 0 ${base_height/2}" rpy="0 0 0" />
+            <material name="blue" />
+        </collision>
+        <xacro:box_inertia m="5.0" l="${base_length}" w="${base_width}" h="${base_height}"
                            xyz="0 0 ${base_height/2.0}" rpy="0 0 0" />
     </link>
@@ -27,6 +34,13 @@
                 <material name="grey" />
             </visual>
-            <xacro:box_inertia m="1.0" r="${wheel_radius}" l="wheel_length"
-                            xyz="0 0 0" rpy="${pi/2.0} 0 0" />
+            <collision>
+                <geometry>
+                    <cylinder radius="${wheel_radius}" length="${wheel_length}" />
+                </geometry>
+                <origin xyz="0 0 0" rpy="${pi/2.0} 0 0" />
+                <material name="grey" />
+            </collision>
+            <xacro:cylinder_inertia m="1.0" r="${wheel_radius}" l="${base_height}"
+                                    xyz="0 0 0" rpy="${pi/2.0} 0 0" />
         </link>
     </xacro:macro>
@@ -41,6 +55,13 @@
             <material name="grey" />
         </visual>
-        <xacro:box_inertia m="0.5" r="${wheel_radius/2.0}"
-                xyz="0 0 0" rpy="0 0 0" />
+        <collision>
+            <geometry>
+                <sphere radius="${wheel_radius/2.0}" />
+            </geometry>
+            <origin xyz="0 0 0" rpy="0 0 0" />
+            <material name="grey" />
+        </collision>
+        <xacro:sphere_inertia m="0.5" r="${wheel_radius/2.0}"
+                              xyz="0 0 0" rpy="0 0 0" />
     </link>
     <joint name="base_joint" type="fixed">

Commit message: last changes

File: src/my_robot_description/urdf/common_properties.xacro (robot description, xacro)
@@ -4,4 +4,10 @@
     <material name="blue">
         <color rgba="${blue_color}" />
+    </material>
+    <material name="orange">
+        <color rgba="1 0.7 0 1" />
+    </material>
+    <material name="yellow">
+        <color rgba="0.5 0.7 0 1" />
     </material>
     <material name="grey">
