Commit message: last changes

File: src/my_robot_description/urdf/arm.xacro (robot description, xacro)
@@ -1,52 +1,77 @@
 <?xml version="1.0"?>
 <robot xmlns:xacro="http://www.ros.org/wiki/xacro">
-    <link name="base_footprint" />
+    <xacro:property name="arm_base_length" value="0.1" />
+    <xacro:property name="arm_base_width" value="0.1" />
+    <xacro:property name="arm_base_height" value="0.02" />
+    <xacro:property name="forearm_radius" value="0.02" />
+    <xacro:property name="forearm_length" value="0.3" />
+    <xacro:property name="hand_radius" value="0.02" />
+    <xacro:property name="hand_length" value="0.3" />
     <link name="arm_base_link">
         <visual>
             <geometry>
-                <box size="0.1 0.1 0.02" />
+                <box size="${arm_base_length} ${arm_base_width} ${arm_base_height}" />
             </geometry>
-            <origin xyz="0 0 0" rpy="0 0 0" />
+            <origin xyz="0 0 ${arm_base_height / 2.0}" rpy="0 0 0" />
             <material name="orange" />
         </visual>
         <collision>
             <geometry>
-                <box size="0.1 0.1 0.02" />
+                <box size="${arm_base_length} ${arm_base_width} ${arm_base_height}" />
             </geometry>
-            <origin xyz="0 0 0" rpy="0 0 0" />
-            <material name="orange" />
+            <origin xyz="0 0 ${arm_base_height / 2.0}" rpy="0 0 0" />
         </collision>
-        <xacro:box_inertia m="0.5" l="0.1" w="0.1" h="0.02"
-                           xyz="0 0 0" rpy="0 0 0" />
+        <xacro:box_inertia m="0.5" l="${2*arm_base_length}" w="${2*arm_base_width}" h="${2*arm_base_height}"
+                           xyz="0 0 ${arm_base_height / 2.0}" rpy="0 0 0" />
     </link>
     <link name="forearm_link">
         <visual>
             <geometry>
-                <cylinder radius="0.02" length="0.3" />
+                <cylinder radius="${forearm_radius}" length="${forearm_length}" />
             </geometry>
-            <origin xyz="0 0 0.15" rpy="0 0 0" />
+            <origin xyz="0 0 ${forearm_length / 2.0}" rpy="0 0 0" />
+            <material name="yellow" />
+        </visual>
+        <collision>
+            <geometry>
+                <cylinder radius="${forearm_radius}" length="${forearm_length}" />
+            </geometry>
+            <origin xyz="0 0 ${forearm_length / 2.0}" rpy="0 0 0" />
+        </collision>
+        <xacro:cylinder_inertia m="0.3" r="${2*forearm_radius}" h="${2*forearm_length}"
+                                xyz="0 0 ${forearm_length / 2.0}" rpy="0 0 0" />
+    </link>
+    <link name="hand_link">
+        <visual>
+            <geometry>
+                <cylinder radius="${hand_radius}" length="${hand_length}" />
+            </geometry>
+            <origin xyz="0 0 ${hand_length / 2.0}" rpy="0 0 0" />
             <material name="orange" />
         </visual>
         <collision>
-            <geometry>
-                <cylinder radius="0.02" length="0.3" />
+             <geometry>
+                <cylinder radius="${hand_radius}" length="${hand_length}" />
             </geometry>
-            <origin xyz="0 0 0.15" rpy="0 0 0" />
-            <material name="orange" />
+            <origin xyz="0 0 ${hand_length / 2.0}" rpy="0 0 0" />
         </collision>
-        <xacro:cylinder_inertia m="0.3" r="0.02" l="0.3"
-                           xyz="0 0 0" rpy="0 0 0" />
+        <xacro:cylinder_inertia m="0.3" r="${2*hand_radius}" h="${2*hand_length}"
+                                xyz="0 0 ${hand_length / 2.0}" rpy="0 0 0" />
     </link>
-    <joint name="arm_base_link_base_footprint_joint" type="fixed">
-        <parent link="base_footprint" />
-        <child link="arm_base_link" />
-        <origin xyz="0 0 0" rpy="0 0 0"/>
-    </joint>
-    <joint name="forearm_base_joint" type="revolute">
+    <joint name="arm_base_forearm_joint" type="revolute">
         <parent link="arm_base_link" />
         <child link="forearm_link" />
-        <origin xyz="0 0 1" rpy="0 0 0"/>
-        <axis xyz="1 0 0" />
-        <limit lower="${-pi/2}" upper="${pi/2}" effort="10" velocity="10" />
+        <origin xyz="0 0 ${arm_base_height}" rpy="0 0 0" />
+        <axis xyz="0 1 0" />
+        <limit lower="0" upper="${pi/2}" effort="100" velocity="100" />
+        <dynamics friction="0.05" damping="0.1" />
+    </joint>
+    <joint name="forearm_hand_joint" type="revolute">
+        <parent link="forearm_link" />
+        <child link="hand_link" />
+        <origin xyz="0 0 ${forearm_length}" rpy="0 0 0" />
+        <axis xyz="0 1 0" />
+        <limit lower="0" upper="${pi/2}" effort="100" velocity="100" />
+        <dynamics friction="0.05" damping="0.1" />
     </joint>
 </robot>

File: src/my_robot_description/urdf/common_properties.xacro (robot description, xacro)
@@ -1,16 +1,15 @@
 <?xml version="1.0"?>
 <robot xmlns:xacro="http://www.ros.org/wiki/xacro">
-    <xacro:property name="blue_color" value="0 0 0.5 1" />
     <material name="blue">
-        <color rgba="${blue_color}" />
-    </material>
-    <material name="orange">
-        <color rgba="1 0.7 0 1" />
-    </material>
-    <material name="yellow">
-        <color rgba="0.5 0.7 0 1" />
+        <color rgba="0 0 0.5 1" />
     </material>
     <material name="grey">
         <color rgba="0.5 0.5 0.5 1" />
+    </material>
+    <material name="orange">
+        <color rgba="1.0 0.5 0 1" />
+    </material>
+    <material name="yellow">
+        <color rgba="1.0 1.0 0 1" />
     </material>
     <xacro:macro name="box_inertia" params="m l w h xyz rpy">
@@ -20,14 +19,14 @@
             <inertia ixx="${(m/12) * (h*h + l*l)}" ixy="0" ixz="0"
                      iyy="${(m/12) * (w*w + l*l)}" iyz="0"
-                     izz="${m/12*(w*w + h*h)}" />
+                     izz="${(m/12) * (w*w + h*h)}" />
         </inertial>
     </xacro:macro>
-    <xacro:macro name="cylinder_inertia" params="m r l xyz rpy">
+    <xacro:macro name="cylinder_inertia" params="m r h xyz rpy">
         <inertial>
             <origin xyz="${xyz}" rpy="${rpy}" />
             <mass value="${m}" />
-            <inertia ixx="${m/12*(3*r*r + l*l)}" ixy="0" ixz="0"
-                     iyy="${m/12*(3*r*r + l*l)}" iyz="0"
-                     izz="${m/12*(r*r)}" />
+            <inertia ixx="${(m/12) * (3*r*r + h*h)}" ixy="0" ixz="0"
+                     iyy="${(m/12) * (3*r*r + h*h)}" iyz="0"
+                     izz="${(m/2) * (r*r)}" />
         </inertial>
     </xacro:macro>
@@ -37,6 +36,6 @@
             <mass value="${m}" />
             <inertia ixx="${(2/5) * m * r * r}" ixy="0" ixz="0"
-                     iyy="${(2/5)*m*r*r}" iyz="0"
-                     izz="${(2/5)*m*r*r}" />
+                     iyy="${(2/5) * m * r * r}" iyz="0"
+                     izz="${(2/5) * m * r * r}" />
         </inertial>
     </xacro:macro>

File: src/my_robot_description/urdf/mobile_base.xacro (robot description, xacro)
@@ -2,5 +2,5 @@
 <robot xmlns:xacro="http://www.ros.org/wiki/xacro">
     <xacro:property name="base_length" value="0.6" />
-    <xacro:property name="base_width" value="0.5" />
+    <xacro:property name="base_width" value="0.4" />
     <xacro:property name="base_height" value="0.2" />
     <xacro:property name="wheel_radius" value="0.1" />
@@ -12,5 +12,5 @@
                 <box size="${base_length} ${base_width} ${base_height}" />
             </geometry>
-            <origin xyz="0 0 ${base_height/2}" rpy="0 0 0" />
+            <origin xyz="0 0 ${base_height / 2.0}" rpy="0 0 0" />
             <material name="blue" />
         </visual>
@@ -19,9 +19,8 @@
                 <box size="${base_length} ${base_width} ${base_height}" />
             </geometry>
-            <origin xyz="0 0 ${base_height/2}" rpy="0 0 0" />
-            <material name="blue" />
+            <origin xyz="0 0 ${base_height / 2.0}" rpy="0 0 0" />
         </collision>
         <xacro:box_inertia m="5.0" l="${2*base_length}" w="${2*base_width}" h="${2*base_height}"
-                           xyz="0 0 ${base_height/2.0}" rpy="0 0 0" />
+                           xyz="0 0 ${base_height / 2.0}" rpy="0 0 0" />
     </link>
     <xacro:macro name="wheel_link" params="prefix">
@@ -31,5 +30,5 @@
                     <cylinder radius="${wheel_radius}" length="${wheel_length}" />
                 </geometry>
-                <origin xyz="0 0 0" rpy="${pi/2.0} 0 0" />
+                <origin xyz="0 0 0" rpy="${pi / 2.0} 0 0" />
                 <material name="grey" />
             </visual>
@@ -38,9 +37,8 @@
                     <cylinder radius="${wheel_radius}" length="${wheel_length}" />
                 </geometry>
-                <origin xyz="0 0 0" rpy="${pi/2.0} 0 0" />
-                <material name="grey" />
+                <origin xyz="0 0 0" rpy="${pi / 2.0} 0 0" />
             </collision>
-            <xacro:cylinder_inertia m="1.0" r="${2*wheel_radius}" l="${2*base_height}"
-                                    xyz="0 0 0" rpy="${pi/2.0} 0 0" />
+            <xacro:cylinder_inertia m="1.0" r="${2*wheel_radius}" h="${2*wheel_length}"
+                                    xyz="0 0 0" rpy="${pi / 2.0} 0 0" />
         </link>
     </xacro:macro>
@@ -50,5 +48,5 @@
         <visual>
             <geometry>
-                <sphere radius="${wheel_radius/2.0}" />
+                <sphere radius="${wheel_radius / 2.0}" />
             </geometry>
             <origin xyz="0 0 0" rpy="0 0 0" />
@@ -57,10 +55,9 @@
         <collision>
             <geometry>
-                <sphere radius="${wheel_radius/2.0}" />
+                <sphere radius="${wheel_radius / 2.0}" />
             </geometry>
             <origin xyz="0 0 0" rpy="0 0 0" />
-            <material name="grey" />
         </collision>
-        <xacro:sphere_inertia m="0.5" r="${2*wheel_radius/2.0}"
+        <xacro:sphere_inertia m="0.5" r="${2*wheel_radius / 2.0}"
                               xyz="0 0 0" rpy="0 0 0" />
     </link>
@@ -68,10 +65,10 @@
         <parent link="base_footprint" />
         <child link="base_link" />
-        <origin xyz="0 0 ${base_height/2}" rpy="0 0 0"/>
+        <origin xyz="0 0 ${wheel_radius}" rpy="0 0 0"/>
     </joint>
     <joint name="base_right_wheel_joint" type="continuous">
         <parent link="base_link" />
         <child link="right_wheel_link" />
-        <origin xyz="${-base_length / 4.0} ${(base_width + wheel_length)/2} 0" rpy="0 0 0" />
+        <origin xyz="${-base_length / 4.0} ${-(base_width + wheel_length) / 2.0} 0" rpy="0 0 0" />
         <axis xyz="0 1 0" />
     </joint>
@@ -79,5 +76,5 @@
         <parent link="base_link" />
         <child link="left_wheel_link" />
-        <origin xyz="${-base_length / 4.0} ${-(base_width + wheel_length)/2} 0" rpy="0 0 0" />
+        <origin xyz="${-base_length / 4.0} ${(base_width + wheel_length) / 2.0} 0" rpy="0 0 0" />
         <axis xyz="0 1 0" />
     </joint>
@@ -85,5 +82,5 @@
         <parent link="base_link" />
         <child link="caster_wheel_link" />
-        <origin xyz="${base_length / 3.0} 0 ${-wheel_radius/2}" rpy="0 0 0" />
+        <origin xyz="${base_length / 3.0} 0 ${-wheel_radius / 2.0}" rpy="0 0 0" />
     </joint>
 </robot>

File: src/my_robot_description/urdf/mobile_base_gazebo.xacro (robot description, xacro)
@@ -5,8 +5,8 @@
     </gazebo>
     <gazebo reference="right_wheel_link">
-        <material>Gazebo/Black</material>
+        <material>Gazebo/Grey</material>
     </gazebo>
     <gazebo reference="left_wheel_link">
-        <material>Gazebo/Black</material>
+        <material>Gazebo/Grey</material>
     </gazebo>
     <gazebo reference="caster_wheel_link">
@@ -26,10 +26,10 @@
             <wheel_diameter>0.2</wheel_diameter>
             <!-- output -->
-            <publish_odom>true</publish_odom> <!-- keeps the position of the robot with respect to the initial frame -->
+            <publish_odom>true</publish_odom>
             <publish_odom_tf>true</publish_odom_tf>
             <publish_wheel_tf>true</publish_wheel_tf>
             <odometry_topic>odom</odometry_topic>
             <odometry_frame>odom</odometry_frame>
-            <robot_base_frame>base_footprint</robot_base_frame> <!-- base frame of the robot -->
+            <robot_base_frame>base_footprint</robot_base_frame>
         </plugin>
     </gazebo>

File: src/my_robot_description/urdf/my_robot.urdf.xacro (robot description, xacro)
@@ -4,4 +4,11 @@
     <xacro:include filename="mobile_base.xacro" />
     <xacro:include filename="mobile_base_gazebo.xacro" />
-    <xacro:include filename="camera.xacro" />
+    <xacro:include filename="arm.xacro" />
+    <xacro:include filename="arm_gazebo.xacro" />
+    <joint name="mobile_base_arm_joint" type="fixed">
+        <parent link="base_link" />
+        <child link="arm_base_link" />
+        <origin xyz="${base_length / 4.0} 0 ${base_height}" rpy="0 0 0" />
+    </joint>
+    <!-- <xacro:include filename="camera.xacro" /> -->
 </robot>

File: src/my_robot_description/urdf/standalone_arm.urdf.xacro (robot description, xacro)
@@ -2,4 +2,7 @@
 <robot name="my_robot" xmlns:xacro="http://www.ros.org/wiki/xacro">
     <xacro:include filename="common_properties.xacro" />
+    <xacro:include filename="mobile_base.xacro" />
+    <xacro:include filename="mobile_base_gazebo.xacro" />
     <xacro:include filename="arm.xacro" />
+    <xacro:include filename="arm_gazebo.xacro" />
 </robot>
